Commit message: Removed unnecessary components

File: rotors_description/urdf/component_snippets.xacro (robot description, xacro)
@@ -762,5 +762,5 @@
   <xacro:macro name="ground_truth_imu_and_odometry" params="namespace parent_link">
     <!-- Mount an IMU providing ground truth. -->
-    <xacro:imu_plugin_macro
+    <!-- <xacro:imu_plugin_macro
       namespace="${namespace}"
       imu_suffix="gt"
@@ -778,5 +778,5 @@
       <inertia ixx="0.00001" ixy="0.0" ixz="0.0" iyy="0.00001" iyz="0.0" izz="0.00001" />
       <origin xyz="0 0 0" rpy="0 0 0" />
-    </xacro:imu_plugin_macro>
+    </xacro:imu_plugin_macro> -->
     <!-- Mount a generic odometry sensor providing ground truth. -->
     <xacro:odometry_plugin_macro

File: rotors_description/urdf/f450_base.xacro (robot description, xacro)
@@ -22,20 +22,6 @@
   <!-- Instantiate a controller. -->
   <xacro:controller_plugin_macro namespace="${namespace}" imu_sub_topic="imu" />
-  <xacro:if value="$(arg enable_mavlink_interface)">
-    <!-- Instantiate mavlink telemetry interface. -->
-    <xacro:default_mavlink_interface namespace="${namespace}" imu_sub_topic="imu" rotor_count="4" />
-  </xacro:if>
-  <!-- Mount an ADIS16448 IMU. -->
-  <xacro:default_imu namespace="${namespace}" parent_link="${namespace}/base_link" />
   <xacro:if value="$(arg enable_ground_truth)">
     <xacro:ground_truth_imu_and_odometry namespace="${namespace}" parent_link="${namespace}/base_link" />
   </xacro:if>
-  <xacro:if value="$(arg enable_logging)">
-    <!-- Instantiate a logger -->
-    <xacro:bag_plugin_macro
-      namespace="${namespace}"
-      bag_file="$(arg log_file)"
-      rotor_velocity_slowdown_sim="${rotor_velocity_slowdown_sim}"
-      wait_to_record_bag="$(arg wait_to_record_bag)" />
-  </xacro:if>
 </robot>

File: rotors_description/urdf/multirotor_base.xacro (robot description, xacro)
@@ -57,10 +57,4 @@
         </geometry>
       </visual>
-      <collision>
-        <origin xyz="0 0 0" rpy="0 0 0" />
-        <geometry>
-          <box size="${body_width} ${body_width} ${body_height}" /> <!-- [m] [m] [m] -->
-        </geometry>
-      </collision>
     </link>
     <!-- attach multirotor_base_plugin to the base_link -->
@@ -103,9 +97,4 @@
         </geometry>
       </visual>
-      <collision>
-        <geometry>
-          <cylinder length="0.005" radius="${radius_rotor}" /> <!-- [m] -->
-        </geometry>
-      </collision>
     </link>
     <gazebo>
