Commit message: Model with quad and ball
Add single quadrotor and ball model with a floating joint
Restore quadrotor collisions
Restore ground plane and world update rate

File: rotors_description/urdf/multirotor_base.xacro (robot description, xacro)
@@ -57,4 +57,10 @@
         </geometry>
       </visual>
+      <collision>
+        <origin xyz="0 0 0" rpy="0 0 0" />
+        <geometry>
+          <box size="${body_width} ${body_width} ${body_height}" /> <!-- [m] [m] [m] -->
+        </geometry>
+      </collision>
     </link>
     <!-- attach multirotor_base_plugin to the base_link -->
@@ -97,4 +103,9 @@
         </geometry>
       </visual>
+      <collision>
+        <geometry>
+          <cylinder length="0.005" radius="${radius_rotor}" /> <!-- [m] -->
+        </geometry>
+      </collision>
     </link>
     <gazebo>
