Commit message: Cable plugin [WIP]

File: rotors_description/urdf/ball.xacro (robot description, xacro)
@@ -1,5 +1,5 @@
 <?xml version="1.0"?>
 <robot xmlns:xacro="http://ros.org/wiki/xacro">
-  <xacro:macro name="ball_macro" params="namespace parent_link ball_radius ball_weight *origin">
+  <xacro:macro name="ball_macro" params="namespace parent_link ball_radius ball_weight cable_length parent_frame_id child_frame_id *origin">
     <link name="${namespace}/ball_link">
       <inertial>
@@ -25,10 +25,22 @@
       </collision>
     </link>
-    <joint name="${namespace}_cable_joint" type="floating">
+    <joint name="${namespace}/ball_joint" type="fixed">
       <xacro:insert_block name="origin" />
       <parent link="${parent_link}" />
       <child link="${namespace}/ball_link" />
     </joint>
-    <gazebo reference="ball">
+    <gazebo>
+      <plugin name="${namespace}_cable_plugin" filename="librotors_gazebo_cable_plugin.so">
+        <robotNamespace>${namespace}</robotNamespace>
+        <jointName>${namespace}/ball_joint</jointName>
+        <linkName>${namespace}/ball_link</linkName>
+        <ballRadius>${ball_radius}</ballRadius>
+        <ballWeight>${ball_weight}</ballWeight>
+        <cableLength>${cable_length}</cableLength>
+        <parentFrameId>${parent_frame_id}</parentFrameId>
+        <childFrameId>${child_frame_id}</childFrameId>
+      </plugin>
+    </gazebo>
+    <gazebo reference="${namespace}/ball_link">
       <mu1>10</mu1>
       <mu2>10</mu2>

File: rotors_description/urdf/mav_with_ball.xacro (robot description, xacro)
@@ -2,11 +2,14 @@
 <robot name="$(arg mav_name)" xmlns:xacro="http://ros.org/wiki/xacro">
   <!-- Instantiate the mav-->
+  <xacro:include filename="$(find rotors_description)/urdf/$(arg mav_name)_base.xacro" />
   <xacro:include filename="$(find rotors_description)/urdf/ball.xacro" />
-  <xacro:include filename="$(find rotors_description)/urdf/$(arg mav_name)_base.xacro" />
   <xacro:ball_macro
-    namespace="${namespace}/ball"
-    parent_link="${namespace}/base_link"
+    namespace="$(arg mav_name)"
+    parent_link="$(arg mav_name)/base_link"
     ball_radius="0.05"
-    ball_weight="0.1">
+    ball_weight="0.1"
+    cable_length="1.0"
+    parent_frame_id="$(arg mav_name)/base_link"
+    child_frame_id="$(arg mav_name)/ball_link">
     <origin xyz="0.0 0.0 -1.0" rpy="0.0 0.0 0.0" />
   </xacro:ball_macro>

Commit message: Single slungload working with single quadrotor

File: rotors_description/urdf/ball.xacro (robot description, xacro)
@@ -1,11 +1,11 @@
 <?xml version="1.0"?>
 <robot xmlns:xacro="http://ros.org/wiki/xacro">
-  <xacro:macro name="ball_macro" params="namespace parent_link ball_radius ball_weight cable_length parent_frame_id child_frame_id *origin">
+  <xacro:macro name="ball_macro" params="namespace parent_link ball_radius ball_mass cable_length *origin">
     <link name="${namespace}/ball_link">
       <inertial>
-        <mass value="${ball_weight}" />
+        <mass value="${ball_mass}" />
         <!-- center of mass (com) is defined w.r.t. link local coordinate system -->
         <!-- give a little y-offset to make the top precess -->
-        <origin xyz="0 0 0" />
+        <origin xyz="0 0 0" rpy="0 0 0" />
         <inertia  ixx="1" ixy="0.0"  ixz="0.0"  iyy="1"  iyz="0.0"  izz="1" />
       </inertial>
@@ -25,5 +25,5 @@
       </collision>
     </link>
-    <joint name="${namespace}/ball_joint" type="fixed">
+    <joint name="${namespace}/ball_joint" type="floating">
       <xacro:insert_block name="origin" />
       <parent link="${parent_link}" />
@@ -33,11 +33,8 @@
       <plugin name="${namespace}_cable_plugin" filename="librotors_gazebo_cable_plugin.so">
         <robotNamespace>${namespace}</robotNamespace>
-        <jointName>${namespace}/ball_joint</jointName>
+        <parentLinkName>${namespace}/base_link</parentLinkName>
         <linkName>${namespace}/ball_link</linkName>
-        <ballRadius>${ball_radius}</ballRadius>
-        <ballWeight>${ball_weight}</ballWeight>
+        <ballMass>${ball_mass}</ballMass>
         <cableLength>${cable_length}</cableLength>
-        <parentFrameId>${parent_frame_id}</parentFrameId>
-        <childFrameId>${child_frame_id}</childFrameId>
       </plugin>
     </gazebo>

File: rotors_description/urdf/mav_with_ball.xacro (robot description, xacro)
@@ -8,8 +8,6 @@
     parent_link="$(arg mav_name)/base_link"
     ball_radius="0.05"
-    ball_weight="0.1"
+    ball_mass="0.1"
     cable_length="1.0"
-    parent_frame_id="$(arg mav_name)/base_link"
-    child_frame_id="$(arg mav_name)/ball_link">
     <origin xyz="0.0 0.0 -1.0" rpy="0.0 0.0 0.0" />
   </xacro:ball_macro>

Commit message: rviz setup for slungload

File: rotors_description/urdf/ball.xacro (robot description, xacro)
@@ -1,5 +1,5 @@
 <?xml version="1.0"?>
 <robot xmlns:xacro="http://ros.org/wiki/xacro">
-  <xacro:macro name="ball_macro" params="namespace parent_link ball_radius ball_mass cable_length *origin">
+  <xacro:macro name="ball_macro" params="namespace parent_link ball_radius ball_mass cable_length parent_frame_id child_frame_id *origin">
     <link name="${namespace}/ball_link">
       <inertial>
@@ -37,4 +37,6 @@
         <ballMass>${ball_mass}</ballMass>
         <cableLength>${cable_length}</cableLength>
+        <parentFrameId>${parent_frame_id}</parentFrameId>
+        <childFrameId>${child_frame_id}</childFrameId>
       </plugin>
     </gazebo>

File: rotors_description/urdf/mav_with_ball.xacro (robot description, xacro)
@@ -10,4 +10,6 @@
     ball_mass="0.1"
     cable_length="1.0"
+    parent_frame_id="$(arg mav_name)/base_link"
+    child_frame_id="$(arg mav_name)/ball_link">
     <origin xyz="0.0 0.0 -1.0" rpy="0.0 0.0 0.0" />
   </xacro:ball_macro>
